Commit message: add example_track_flipper

File: urdf_xacro/example_track_flipper.urdf.xacro (robot description, xacro)
@@ -22,5 +22,5 @@
     <!-- base_link to be wrapped by the track -->
     <link name="base_link">
-        <xacro:make_box_inertia mass="1" size_x="0.5" size_y="0.325" size_z="0.1" />
+        <xacro:make_box_inertia mass="10" size_x="0.5" size_y="0.325" size_z="0.1" />
         <visual>
             <geometry>
@@ -158,3 +158,139 @@
         <child link="idler_right" />
     </joint>
+    <!-- flipper fl -->
+    <link name="flipper_fl_link">
+    </link>
+    <joint name="flipper_fl_joint" type="continuous">
+        <origin xyz="0.2 0.295 0" rpy="0 0 0" />
+        <parent link="base_link" />
+        <child link="flipper_fl_link" />
+        <axis xyz="0.0 1.0 0.0"/>
+    </joint>
+    <transmission name="flipper_fl_transmission">
+        <type>transmission_interface/SimpleTransmission</type>
+        <joint name="flipper_fl_joint">
+            <hardwareInterface>hardware_interface/EffortJointInterface</hardwareInterface>
+        </joint>
+        <actuator name="flipper_fl_actuator">
+            <mechanicalReduction>1</mechanicalReduction>
+        </actuator>
+    </transmission>
+    <link name="flipper_fl_sprocket">
+        <xacro:make_wheel_inertia mass="0.2" radius="0.064" length="0.1115" />
+        <visual>
+            <origin xyz="0 0 0" rpy="${pi / 2} 0 0" />
+            <geometry>
+                <cylinder radius="0.064" length="0.1115" />
+            </geometry>
+        </visual>
+        <!-- <collision>
+            <origin xyz="0 0 0" rpy="${pi / 2} 0 0" />
+            <geometry>
+                <cylinder radius="0.064" length="0.1115" />
+            </geometry>
+        </collision> -->
+    </link>
+    <joint name="flipper_fl_sprocket_axle" type="continuous">
+        <origin xyz="0.0 0.0 0" rpy="0 0 0" />
+        <parent link="flipper_fl_link" />
+        <child link="flipper_fl_sprocket" />
+        <axis xyz="0.0 1.0 0.0"/>
+    </joint>
+    <transmission name="flipper_fl_sprocket_axle_transmission">
+        <type>transmission_interface/SimpleTransmission</type>
+        <joint name="flipper_fl_sprocket_axle">
+            <hardwareInterface>hardware_interface/VelocityJointInterface</hardwareInterface>
+        </joint>
+        <actuator name="flipper_fl_sprocket_axle_actuator">
+            <mechanicalReduction>1</mechanicalReduction>
+        </actuator>
+    </transmission>
+    <link name="flipper_fl_idler">
+        <xacro:make_wheel_inertia mass="0.2" radius="0.0225" length="0.1115" />
+        <visual>
+            <origin xyz="0 0 0" rpy="${pi / 2} 0 0" />
+            <geometry>
+                <cylinder radius="0.0225" length="0.1115" />
+            </geometry>
+        </visual>
+        <!-- <collision>
+            <origin xyz="0 0 0" rpy="${pi / 2} 0 0" />
+            <geometry>
+                <cylinder radius="0.0225" length="0.1115" />
+            </geometry>
+        </collision> -->
+    </link>
+    <joint name="flipper_fl_idler_axle" type="fixed">
+        <origin xyz="0.26 0.0 0" rpy="0 0 0" />
+        <parent link="flipper_fl_link" />
+        <child link="flipper_fl_idler" />
+    </joint>
+    <!-- flipper fr -->
+    <link name="flipper_fr_link">
+    </link>
+    <joint name="flipper_fr_joint" type="continuous">
+        <origin xyz="0.2 -0.295 0" rpy="0 0 0" />
+        <parent link="base_link" />
+        <child link="flipper_fr_link" />
+        <axis xyz="0.0 1.0 0.0"/>
+    </joint>
+    <transmission name="flipper_fr_transmission">
+        <type>transmission_interface/SimpleTransmission</type>
+        <joint name="flipper_fr_joint">
+            <hardwareInterface>hardware_interface/EffortJointInterface</hardwareInterface>
+        </joint>
+        <actuator name="flipper_fr_actuator">
+            <mechanicalReduction>1</mechanicalReduction>
+        </actuator>
+    </transmission>
+    <link name="flipper_fr_sprocket">
+        <xacro:make_wheel_inertia mass="0.2" radius="0.064" length="0.1115" />
+        <visual>
+            <origin xyz="0 0 0" rpy="${pi / 2} 0 0" />
+            <geometry>
+                <cylinder radius="0.064" length="0.1115" />
+            </geometry>
+        </visual>
+        <!-- <collision>
+            <origin xyz="0 0 0" rpy="${pi / 2} 0 0" />
+            <geometry>
+                <cylinder radius="0.064" length="0.1115" />
+            </geometry>
+        </collision> -->
+    </link>
+    <joint name="flipper_fr_sprocket_axle" type="continuous">
+        <origin xyz="0.0 0.0 0" rpy="0 0 0" />
+        <parent link="flipper_fr_link" />
+        <child link="flipper_fr_sprocket" />
+        <axis xyz="0.0 1.0 0.0"/>
+    </joint>
+    <transmission name="flipper_fr_sprocket_axle_transmission">
+        <type>transmission_interface/SimpleTransmission</type>
+        <joint name="flipper_fr_sprocket_axle">
+            <hardwareInterface>hardware_interface/VelocityJointInterface</hardwareInterface>
+        </joint>
+        <actuator name="flipper_fr_sprocket_axle_actuator">
+            <mechanicalReduction>1</mechanicalReduction>
+        </actuator>
+    </transmission>
+    <link name="flipper_fr_idler">
+        <xacro:make_wheel_inertia mass="0.2" radius="0.0225" length="0.1115" />
+        <visual>
+            <origin xyz="0 0 0" rpy="${pi / 2} 0 0" />
+            <geometry>
+                <cylinder radius="0.0225" length="0.1115" />
+            </geometry>
+        </visual>
+        <!-- <collision>
+            <origin xyz="0 0 0" rpy="${pi / 2} 0 0" />
+            <geometry>
+                <cylinder radius="0.0225" length="0.1115" />
+            </geometry>
+        </collision> -->
+    </link>
+    <joint name="flipper_fr_idler_axle" type="fixed">
+        <origin xyz="0.26 0.0 0" rpy="0 0 0" />
+        <parent link="flipper_fr_link" />
+        <child link="flipper_fr_idler" />
+    </joint>
 </robot>

File: urdf_xacro/example_track_flipper_gazebo.urdf.xacro (robot description, xacro)
@@ -1,6 +1,6 @@
-<robot name="example_track" xmlns:xacro="http://www.ros.org/wiki/xacro">
+<robot name="example_track_flipper" xmlns:xacro="http://www.ros.org/wiki/xacro">
     <!-- -->
     <xacro:include filename="$(find gazebo_continuous_track)/urdf_xacro/macros_track_gazebo.urdf.xacro" />
-    <xacro:include filename="example_track.urdf.xacro" />
+    <xacro:include filename="example_track_flipper.urdf.xacro" />
     <!-- -->
     <xacro:property name="track_material">
@@ -34,4 +34,26 @@
         </pattern>
     </xacro:make_track>
+    <xacro:make_flipper name="flipper_fl" x="0.33" y="0.295" mass="0.4" length="0.26" radius="0.064" dradius="0.0225" pitch="0.14627604" width="0.1115" parent="flipper_fl_link" sprocket_joint="flipper_fl_sprocket_axle" pitch_diameter="0.223">
+        <xacro:insert_block name="track_material" />
+        <pattern>
+            <elements_per_round>40</elements_per_round>
+            <element>
+                <xacro:make_cylinder_element pose="0 0 0.01 ${pi / 2} 0 0" length="0.1115" radius="0.0125">
+                    <xacro:insert_block name="track_material" />
+                </xacro:make_cylinder_element>
+            </element>
+        </pattern>
+    </xacro:make_flipper>
+    <xacro:make_flipper name="flipper_fr" x="0.33" y="-0.295" mass="0.4" length="0.26" radius="0.064" dradius="0.0225" pitch="0.14627604" width="0.1115" parent="flipper_fr_link" sprocket_joint="flipper_fr_sprocket_axle" pitch_diameter="0.223">
+        <xacro:insert_block name="track_material" />
+        <pattern>
+            <elements_per_round>40</elements_per_round>
+            <element>
+                <xacro:make_cylinder_element pose="0 0 0.01 ${pi / 2} 0 0" length="0.1115" radius="0.0125">
+                    <xacro:insert_block name="track_material" />
+                </xacro:make_cylinder_element>
+            </element>
+        </pattern>
+    </xacro:make_flipper>
     <!-- ros_control for gazebo -->
     <gazebo>
